Commit message: add example joint urdf element

File: example.urdf.xacro (robot description, xacro)
@@ -10,2 +10,7 @@
   </visual>
 </link>
+<joint name="joint1">
+  <parent link="joint4"/>
+  <child link="jointparent"/>
+  <origin xyz="0 0 0" rpy="0 0 0"/>
+</joint>

Commit message: clean spacing

File: example.urdf.xacro (robot description, xacro)
@@ -5,7 +5,7 @@
       <box size="0.4 5 4" rpy="0 0 0"/>
     </geometry>
-	<material name="red">
-	  <color rgba="0.5 0.7 0.1 1"/>
-	</material>
+	  <material name="red">
+	    <color rgba="0.5 0.7 0.1 1"/>
+	  </material>
   </visual>
 </link>
